Commit message: Collision and inertial properties were added

File: src/medical_rover_description/urdf/chassis.xacro (robot description, xacro)
@@ -12,4 +12,11 @@
                 </material>
             </visual>
+            <collision>
+                <origin xyz="0 0 ${body_height/2}" rpy="0 0 0"/>
+                <geometry>
+                    <box size="${body_length} ${body_width} ${body_height}" />
+                </geometry>
+            </collision>
+            <xacro:box_inertia mass="${body_mass}" x="${body_length}" y="${body_width}" z="${body_height}"/>
         </link>
         <joint name="base_to_chassis" type="fixed">
@@ -19,3 +26,29 @@
         </joint>
     </xacro:macro>
+    <xacro:macro name="caster">
+        <link name="caster_wheel_link">
+            <visual>
+                <origin xyz="0 0 0" rpy="0 0 0"/>
+                <geometry>
+                    <sphere radius="${sphere_radius}" />
+                </geometry>
+                <material name="grey">
+                    <color rgba="0.7 0.7 0.7 1" />
+                </material>
+            </visual>
+        <collision>
+            <origin xyz="0 0 0" rpy="0 0 0"/>
+            <geometry>
+                <sphere radius="${sphere_radius}" />
+            </geometry>
+        </collision>
+        <xacro:sphere_inertia mass="${caster_mass}" radius="${sphere_radius}"/>
+        </link>
+        <joint name="caster_wheel_joint" type="fixed">
+            <parent link="chassis_link"/>
+            <child link="caster_wheel_link"/>
+            <origin xyz="${(body_length/2)-sphere_radius} 0 -${sphere_radius}" rpy="0 0 0"/>
+        </joint>
+>
+    </xacro:macro>
 </robot>

File: src/medical_rover_description/urdf/medical_rover.urdf.xacro (robot description, xacro)
@@ -5,4 +5,5 @@
     <xacro:include filename="chassis.xacro" />
     <xacro:include filename="sensors.xacro" />
+    <xacro:include filename="inertial_values.xacro" />
     <link name="base_link"/>
     <xacro:chassis/>
@@ -11,19 +12,4 @@
     <xacro:lidar/>
     <xacro:camera/>
-    <link name="caster_wheel_link">
-        <visual>
-            <origin xyz="0 0 0" rpy="0 0 0"/>
-            <geometry>
-                <sphere radius="${sphere_radius}" />
-            </geometry>
-            <material name="grey">
-                <color rgba="0.7 0.7 0.7 1" />
-            </material>
-        </visual>
-    </link>
-    <joint name="caster_wheel_joint" type="fixed">
-        <parent link="chassis_link"/>
-        <child link="caster_wheel_link"/>
-        <origin xyz="${(body_length/2)-sphere_radius} 0 -${sphere_radius}" rpy="0 0 0"/>
-    </joint>
+    <xacro:caster/>
 </robot>

File: src/medical_rover_description/urdf/properties.xacro (robot description, xacro)
@@ -1,16 +1,26 @@
 <?xml version="1.0"?>
 <robot xmlns:xacro="http://www.ros.org/wiki/xacro">
+    <!--CHASSIS PROPERTIES-->
     <xacro:property name="body_length" value="0.40" />
     <xacro:property name="body_width" value="0.30" />
     <xacro:property name="body_height" value="0.12" />
+    <xacro:property name="body_mass" value="2.5"/>
+    <!--WHEEL PROPERTIES-->
     <xacro:property name="wheel_radius" value="0.05" />
     <xacro:property name="wheel_width" value="0.03" />
+    <xacro:property name="wheel_mass" value="0.20" />
     <xacro:property name="wheel_x" value="-0.10" />
     <xacro:property name="wheel_y" value="${body_width/2 + wheel_width/2}" />
+    <!--LIDAR PROPERTIES-->
     <xacro:property name="lidar_radius" value="0.03" />
     <xacro:property name="lidar_height" value="0.03" />
+    <xacro:property name="lidar_mass" value="0.10" />
+    <!--CAMERA PROPERTIES-->
     <xacro:property name="camera_length" value="0.04" />
     <xacro:property name="camera_width" value="0.03" />
     <xacro:property name="camera_height" value="0.02" />
+    <xacro:property name="camera_mass" value="0.08" />
+    <!--CASTER WHEEL PROPERTIES-->
     <xacro:property name="sphere_radius" value="0.025" />
+    <xacro:property name="caster_mass" value="0.05" />
 </robot>

File: src/medical_rover_description/urdf/sensors.xacro (robot description, xacro)
@@ -12,4 +12,11 @@
                 </material>
             </visual>
+            <collision>
+                <origin xyz = "0 0 0" rpy = "0 0 0"/>
+                <geometry>
+                    <cylinder radius="${lidar_radius}" length="${lidar_height}" />
+                </geometry>
+            </collision>
+            <xacro:cylinder_inertia mass="${lidar_mass}" radius="${lidar_radius}" length="${lidar_height}"/>
         </link>
         <joint name="lidar_joint" type="fixed">
@@ -30,4 +37,11 @@
                 </material>
             </visual>
+            <collision>
+                <origin xyz="0 0 0" rpy="0 0 0"/>
+                <geometry>
+                    <box size="${camera_width} ${camera_length} ${camera_height}" />
+                </geometry>
+            </collision>
+            <xacro:box_inertia mass="${camera_mass}" x="${camera_width}" y="${camera_length}" z="${camera_height}" />
     </link>
         <joint name="camera_joint" type="fixed">

File: src/medical_rover_description/urdf/wheels.xacro (robot description, xacro)
@@ -12,4 +12,11 @@
                 </material>
             </visual>
+            <collision>
+                <origin xyz="0 0 0" rpy="0 0 0"/>
+                <geometry>
+                    <cylinder radius="${wheel_radius}" length="${wheel_width}" />
+                </geometry>
+            </collision>
+            <xacro:cylinder_inertia mass="${wheel_mass}" radius="${wheel_radius}" length="${wheel_width}"/>
         </link>
         <joint name="${prefix}_wheel_joint" type="continuous">
