Commit message: Implement Gazebo simulation with differential drive controller

File: src/medical_rover_description/urdf/gazebo.xacro (robot description, xacro)
@@ -1,3 +1,9 @@
 <?xml version="1.0"?>
 <robot xmlns:xacro="http://www.ros.org/wiki/xacro">
+    <gazebo>
+        <plugin name="gazebo_ros2_control"
+                filename="libgazebo_ros2_control.so">
+            <parameters>/home/saiyyam/medical_rover_ws/src/medical_rover_gazebo/config/controllers.yaml</parameters>
+        </plugin>
+    </gazebo>
 </robot>

File: src/medical_rover_description/urdf/medical_rover.urdf.xacro (robot description, xacro)
@@ -7,4 +7,5 @@
     <xacro:include filename="inertial_values.xacro" />
     <xacro:include filename="gazebo.xacro"/>
+    <xacro:include filename="ros2_control.xacro"/>
     <link name="base_link"/>
     <xacro:chassis/>
@@ -14,3 +15,4 @@
     <xacro:camera/>
     <xacro:caster/>
+    <xacro:ros2_control/>
 </robot>

File: src/medical_rover_description/urdf/wheels.xacro (robot description, xacro)
@@ -24,5 +24,5 @@
             <child link="${prefix}_wheel_link"/>
             <origin xyz="${wheel_x} ${y_pos} 0" rpy="-${pi/2} 0 0"/>
-            <axis xyz="0 0 -1"/>
+            <axis xyz="0 0 1"/>
         </joint>
     </xacro:macro>
